Commit message: adding moveit2

File: ros_ws/src/cr5_description/urdf/cr5.urdf.xacro (robot description, xacro)
@@ -4,4 +4,5 @@
     <!-- Include common utility macros -->
     <xacro:include filename="$(find cr5_description)/urdf/utils.xacro" />
+    <xacro:include filename="$(find cr5_description)/urdf/ros2control.xacro" />
     <!-- Define common properties -->
     <xacro:property name="mesh_path" value="package://cr5_description/meshes" />
@@ -31,5 +32,5 @@
         <child link="Link1" />
         <axis xyz="0 0 1" />
-        <limit lower="-3.14" upper="3.14" effort="0" velocity="0" />
+        <limit lower="-3.14" upper="3.14" effort="100" velocity="1.0" />
     </joint>
     <!-- Link2 -->
@@ -44,5 +45,5 @@
         <child link="Link2" />
         <axis xyz="0 0 1" />
-        <limit lower="-3.14" upper="3.14" effort="0" velocity="0" />
+        <limit lower="-3.14" upper="3.14" effort="100" velocity="1.0" />
     </joint>
     <!-- Link3 -->
@@ -57,5 +58,5 @@
         <child link="Link3" />
         <axis xyz="0 0 1" />
-        <limit lower="-2.86" upper="2.86" effort="0" velocity="0" />
+        <limit lower="-2.86" upper="2.86" effort="100" velocity="1.0" />
     </joint>
     <!-- Link4 -->
@@ -70,5 +71,5 @@
         <child link="Link4" />
         <axis xyz="0 0 1" />
-        <limit lower="-3.14" upper="3.14" effort="0" velocity="0" />
+        <limit lower="-3.14" upper="3.14" effort="100" velocity="1.0" />
     </joint>
     <!-- Link5 -->
@@ -83,5 +84,5 @@
         <child link="Link5" />
         <axis xyz="0 0 1" />
-        <limit lower="-3.14" upper="3.14" effort="0" velocity="0" />
+        <limit lower="-3.14" upper="3.14" effort="100" velocity="1.0" />
     </joint>
     <!-- Link6 -->
@@ -96,5 +97,5 @@
         <child link="Link6" />
         <axis xyz="0 0 1" />
-        <limit lower="-6.28" upper="6.28" effort="0" velocity="0" />
+        <limit lower="-6.28" upper="6.28" effort="100" velocity="1.0" />
     </joint>
     <!-- GRIPPERS -->

Commit message: basic working with moveit2, feedback issue

File: ros_ws/src/cr5_description/urdf/cr5.urdf.xacro (robot description, xacro)
@@ -100,14 +100,14 @@
     </joint>
     <!-- GRIPPERS -->
-    <!-- <link name="cr5_gripper_link">
-        <xacro:default_visual mesh_filename="${mesh_path}/g_body.dae" material_rgba="${default_material_rgba}" />
-        <xacro:default_collision mesh_filename="${mesh_path}/g_body.dae" />
+    <link name="cr5_gripper_link">
+        <xacro:default_visual mesh_filename="${mesh_path}/gripper.dae" material_rgba="${default_material_rgba}" />
+        <xacro:default_collision mesh_filename="${mesh_path}/gripper.dae" />
     </link>
     <joint name="cr5_gripper_joint" type="fixed">
-        <origin xyz="0 0 -0.002" rpy="0 0 0" />
+        <origin xyz="0 0 0" rpy="0 0 0" />
         <parent link="Link6" />
         <child link="cr5_gripper_link" />
     </joint>
-    <link name="cr5_gripper_left">
+    <!-- <link name="cr5_gripper_left">
         <xacro:default_inertial xyz="5.0777E-11 9.3774E-05 -0.019285" rpy="0 0 0" mass="0.15789" ixx="7.8045E-05" ixy="6.1582E-15" ixz="6.2471E-14" iyy="7.9168E-05" iyz="-1.3822E-07" izz="0.00012951" />
         <xacro:default_visual mesh_filename="${mesh_path}/g_left.dae" material_rgba="${default_material_rgba}" />
